File: diseños de kicad/12Board-PLC4UNI-G1W/out_npn2_opto.kicad_sch (KiCad schematic)
At the start: 3 parts

Commit message: actualizacion 3
Connections:
- net +3.3V is gone; now on net IN: R33.2
- net GND: now also OC7.2
- net IN: no longer OC7.2
Other:
- moved on the sheet: R33
Changed lines of the file:
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@@
 	(wire
 		(pts
-			(xy 125.73 76.2) (xy 125.73 78.74)
+			(xy 125.73 100.33) (xy 125.73 106.68)
+		)
+		(stroke
+			(width 0)
+			(type default)
+		)
+	)
+	(wire
+		(pts
+			(xy 125.73 90.17) (xy 125.73 88.9)
+		)
+		(stroke
+			(width 0)
+			(type default)
+		)
+	)
+	(wire
+		(pts
+			(xy 109.22 88.9) (xy 116.84 88.9)
 		)
 		(stroke
@@
 	(wire
 		(pts
-			(xy 113.03 104.14) (xy 125.73 104.14)
-		)
-		(stroke
-			(width 0)
-			(type default)
-		)
-	)
-	(wire
-		(pts
-			(xy 125.73 104.14) (xy 125.73 100.33)
+			(xy 125.73 88.9) (xy 124.46 88.9)
 		)
 		(stroke
@@
 		(pts
 			(xy 133.35 100.33) (xy 133.35 102.87)
-		)
-		(stroke
-			(width 0)
-			(type default)
-		)
-	)
-	(wire
-		(pts
-			(xy 125.73 86.36) (xy 125.73 90.17)
 		)
 		(stroke
@@
 	(hierarchical_label "IN"
 		(shape input)
-		(at 113.03 104.14 180)
+		(at 109.22 88.9 180)
 		(effects
 			(font
@@
 	)
 	(symbol
-		(lib_id "power:+3.3V")
-		(at 125.73 76.2 0)
+		(lib_id "power:GND")
+		(at 125.73 106.68 0)
 		(unit 1)
 		(exclude_from_sim no)
@@
 		(dnp no)
 		(fields_autoplaced yes)
-		(property "Reference" "#PWR050"
-			(at 125.73 80.01 0)
-			(effects
-				(font
-					(size 1.27 1.27)
-				)
-				(hide yes)
-			)
-		)
-		(property "Value" "+3.3V"
-			(at 125.73 71.12 0)
+		(property "Reference" "#PWR065"
+			(at 125.73 113.03 0)
+			(effects
+				(font
+					(size 1.27 1.27)
+				)
+				(hide yes)
+			)
+		)
+		(property "Value" "GND"
+			(at 125.73 111.76 0)
 			(effects
 				(font
@@
 		)
 		(property "Footprint" ""
-			(at 125.73 76.2 0)
+			(at 125.73 106.68 0)
 			(effects
 				(font
@@
 		)
 		(property "Datasheet" ""
-			(at 125.73 76.2 0)
-			(effects
-				(font
-					(size 1.27 1.27)
-				)
-				(hide yes)
-			)
-		)
-		(property "Description" "Power symbol creates a global label with name \"+3.3V\""
-			(at 125.73 76.2 0)
+			(at 125.73 106.68 0)
+			(effects
+				(font
+					(size 1.27 1.27)
+				)
+				(hide yes)
+			)
+		)
+		(property "Description" "Power symbol creates a global label with name \"GND\" , ground"
+			(at 125.73 106.68 0)
 			(effects
 				(font
@@
 			(project "12Board-PLC4UNI-G1W"
 				(path "/6879a69d-f695-48f8-b9bf-6eca45a0aeb9/dec84266-09cb-480d-928b-b373c3576401/80312332-f227-48d7-8724-587b8d7b3b9a"
-					(reference "#PWR050")
+					(reference "#PWR065")
 					(unit 1)
 				)
@@
 	(symbol
 		(lib_id "Resistor_AKL:R_0603")
-		(at 125.73 82.55 180)
+		(at 120.65 88.9 270)
 		(unit 1)
 		(exclude_from_sim no)
@@
 		(fields_autoplaced yes)
 		(property "Reference" "R33"
-			(at 128.27 81.2799 0)
-			(effects
-				(font
-					(size 1.27 1.27)
-				)
-				(justify right)
+			(at 120.65 82.55 90)
+			(effects
+				(font
+					(size 1.27 1.27)
+				)
 			)
 		)
 		(property "Value" "2.4k"
-			(at 128.27 83.8199 0)
-			(effects
-				(font
-					(size 1.27 1.27)
-				)
-				(justify right)
+			(at 120.65 85.09 90)
+			(effects
+				(font
+					(size 1.27 1.27)
+				)
 			)
 		)
 		(property "Footprint" "Resistor_SMD_AKL:R_0603_1608Metric"
-			(at 125.73 71.12 0)
+			(at 109.22 88.9 0)
 			(effects
 				(font
@@
 		)
 		(property "Datasheet" "~"
-			(at 125.73 82.55 0)
+			(at 120.65 88.9 0)
 			(effects
 				(font
@@
 		)
 		(property "Description" "SMD 0603 Chip Resistor, European Symbol, Alternate KiCad Library"
-			(at 125.73 82.55 0)
-			(effects
-				(font
+			(at 120.65 88.9 0)
+			(effects
+				(font
