File: diseños de kicad/12Board-PLC4UNI-G1W/plc4uni_cpu.kicad_sch (KiCad schematic)
At the start: 4 parts, among them J2 USB_C_Receptacle_USB2.0_14P, U1 ESP32-S3-WROOM-1

Commit message: actualizacion
Connections:
- net ADC_IN_3V3: now also U1.24 (IO47)
- net IN_NPN: now also U1.22 (IO14)
- net IN_NPN1_Opto: now also U1.19 (IO11)
- net IN_NPN2: now also U1.8 (IO15)
- net IN_NPN2_Opto: now also U1.18 (IO10)
- net IN_PNP1: now also U1.12 (IO8)
- net IN_PNP1_Opto: now also U1.21 (IO13)
- net IN_PNP2: now also U1.17 (IO9)
- net IN_PNP2_Opto: now also U1.20 (IO12)
- net NPN_OUT1: now also U1.34 (IO41)
- net NPN_OUT2: now also U1.35 (IO42)
- net OUT_RELAY1: now also U1.32 (IO39)
- net OUT_RELAY2: now also U1.33 (IO40)
- net Opto_NPN: now also U1.30 (IO37)
- net Opto_NPN2: now also U1.31 (IO38)
- net Out_4-20mA: now also U1.26 (IO45)
- net Out_4-20mA_2: now also U1.16 (IO46)
- net PNP_OUT1: now also U1.23 (IO21)
- net PNP_OUT2: now also U1.28 (IO35)
- net PNP_OUT3: now also U1.29 (IO36)
- net SCL: now also U1.27 (IO0)
- net SDA: now also U1.39 (IO1)

Commit message: Actualizacion 48
Connections:
- no-connect marks 0 -> 11
Changed lines of the file:
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@@
 		(color 0 0 0 0)
+	)
+	(no_connect
+		(at 160.02 76.2)
+	)
+	(no_connect
+		(at 129.54 99.06)
+	)
+	(no_connect
+		(at 64.77 82.55)
+	)
+	(no_connect
+		(at 129.54 121.92)
+	)
+	(no_connect
+		(at 64.77 85.09)
+	)
+	(no_connect
+		(at 129.54 96.52)
+	)
+	(no_connect
+		(at 129.54 76.2)
+	)
+	(no_connect
+		(at 129.54 93.98)
+	)
+	(no_connect
+		(at 129.54 88.9)
+	)
+	(no_connect
+		(at 160.02 78.74)
+	)
+	(no_connect
+		(at 129.54 91.44)
 	)
 	(wire
