File: diseños de kicad/12Board-PLC4UNI-G1W/board-plc4uni-G1w.kicad_sch (KiCad schematic)
At the start: 0 parts

Commit message: actu2
Other:
- added sheet fuente (fuente.kicad_sch)
Changed lines of the file:
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@@
+	)
+	(sheet
+		(at 242.57 120.65)
+		(size 25.4 12.7)
+		(exclude_from_sim no)
+		(in_bom yes)
+		(on_board yes)
+		(dnp no)
+		(fields_autoplaced yes)
+		(stroke
+			(width 0.1524)
+			(type solid)
+		)
+		(fill
+			(color 0 0 0 0.0000)
+		)
+		(property "Sheetname" "fuente"
+			(at 242.57 119.9384 0)
+			(effects
+				(font
+					(size 1.27 1.27)
+				)
+				(justify left bottom)
+			)
+		)
+		(property "Sheetfile" "fuente.kicad_sch"
+			(at 242.57 133.9346 0)
+			(effects
+				(font
+					(size 1.27 1.27)
+				)
+				(justify left top)
+			)
+		)
+		(pin "SCLK" bidirectional
+			(at 267.97 124.46 0)
+			(effects
+				(font
+					(size 1.27 1.27)
+				)
+				(justify right)
+			)
+		)
+		(pin "SDA" bidirectional
+			(at 267.97 127 0)
+			(effects
+				(font
+					(size 1.27 1.27)
+				)
+				(justify right)
+			)
+		)
+		(pin "SEL" output
+			(at 267.97 130.81 0)
+			(effects
+				(font
+					(size 1.27 1.27)
+				)
+				(justify right)
+			)
+		)
+		(pin "VOLTAGE_AOUTPUT" output
+			(at 242.57 125.73 180)
+			(effects
+				(font
+					(size 1.27 1.27)
+				)
+				(justify left)
+			)
+		)
+		(instances
+			(project "12Board-PLC4UNI-G1W"
+				(path "/6879a69d-f695-48f8-b9bf-6eca45a0aeb9/dec84266-09cb-480d-928b-b373c3576401"
+					(page "30")
+				)
+			)
+		)
 	)
 	(sheet

Commit message: actualizacion 3
Other:
- added sheet entrada3.3v (entrada3.3v.kicad_sch)
Changed lines of the file:
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@@
+	)
+	(sheet
+		(at 242.57 142.24)
+		(size 29.21 11.43)
+		(exclude_from_sim no)
+		(in_bom yes)
+		(on_board yes)
+		(dnp no)
+		(fields_autoplaced yes)
+		(stroke
+			(width 0.1524)
+			(type solid)
+		)
+		(fill
+			(color 0 0 0 0.0000)
+		)
+		(property "Sheetname" "entrada3.3v"
+			(at 242.57 141.5284 0)
+			(effects
+				(font
+					(size 1.27 1.27)
+				)
+				(justify left bottom)
+			)
+		)
+		(property "Sheetfile" "entrada3.3v.kicad_sch"
+			(at 242.57 154.2546 0)
+			(effects
+				(font
+					(size 1.27 1.27)
+				)
+				(justify left top)
+			)
+		)
+		(pin "+Batt" input
+			(at 242.57 146.05 180)
+			(effects
+				(font
+					(size 1.27 1.27)
+				)
+				(justify left)
+			)
+		)
+		(pin "3.3V" output
+			(at 242.57 149.86 180)
+			(effects
+				(font
+					(size 1.27 1.27)
+				)
+				(justify left)
+			)
+		)
+		(instances
+			(project "12Board-PLC4UNI-G1W"
+				(path "/6879a69d-f695-48f8-b9bf-6eca45a0aeb9/dec84266-09cb-480d-928b-b373c3576401"
+					(page "31")
+				)
+			)
+		)
 	)
 	(sheet

Commit message: actualizacion 47
Other:
- added sheet proteccion24 (proteccion24.kicad_sch)
Changed lines of the file:
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@@
+	(wire
+		(pts
+			(xy 243.84 95.25) (xy 243.84 93.98)
+		)
+		(stroke
+			(width 0)
+			(type default)
+		)
+	)
 	(wire
 		(pts
@@
 	(wire
 		(pts
+			(xy 243.84 93.98) (xy 246.38 93.98)
+		)
+		(stroke
+			(width 0)
+			(type default)
+		)
+	)
+	(wire
+		(pts
 			(xy 191.77 119.38) (xy 187.96 119.38)
 		)
@@
 	(wire
 		(pts
+			(xy 238.76 95.25) (xy 243.84 95.25)
+		)
+		(stroke
+			(width 0)
+			(type default)
+		)
+	)
+	(wire
+		(pts
 			(xy 48.26 123.19) (xy 57.15 123.19)
 		)
@@
 		(pts
 			(xy 83.82 161.29) (xy 83.82 160.02)
+		)
+		(stroke
+			(width 0)
+			(type default)
+		)
+	)
+	(wire
+		(pts
+			(xy 238.76 90.17) (xy 246.38 90.17)
 		)
 		(stroke
@@
 		)
 	)
+	(hierarchical_label "0V-SOURCE"
+		(shape output)
+		(at 238.76 95.25 180)
+		(effects
+			(font
+				(size 1.27 1.27)
+			)
+			(justify right)
+		)
+	)
 	(hierarchical_label "IN_NPN1_Opto"
 		(shape input)
@@
 				(thickness 0.254)
 				(bold yes)
+			)
+			(justify right)
+		)
+	)
+	(hierarchical_label "24V-SOURCE"
+		(shape input)
+		(at 238.76 90.17 180)
+		(effects
+			(font
+				(size 1.27 1.27)
 			)
 			(justify right)
@@
 				)
 			)
+		)
+	)
+	(sheet
+		(at 246.38 87.63)
+		(size 24.13 10.16)
+		(exclude_from_sim no)
+		(in_bom yes)
+		(on_board yes)
+		(dnp no)
+		(fields_autoplaced yes)
+		(stroke
+			(width 0.1524)
+			(type solid)
+		)
+		(fill
+			(color 0 0 0 0.0000)
+		)
+		(property "Sheetname" "proteccion24"
+			(at 246.38 86.9184 0)
+			(effects
+				(font
+					(size 1.27 1.27)
+				)
+				(justify left bottom)
+			)
+		)
+		(property "Sheetfile" "proteccion24.kicad_sch"
+			(at 246.38 98.3746 0)
+			(effects
+				(font
+					(size 1.27 1.27)
+				)
+				(justify left top)
+			)
+		)
+		(pin "+24V" input
+			(at 246.38 90.17 180)
+			(effects
+				(font
+					(size 1.27 1.27)
+				)
+				(justify left)
+			)
+		)
+		(pin "0V" output
+			(at 246.38 93.98 180)
+			(effects
+				(font
+					(size 1.27 1.27)
+				)
+				(justify left)
+			)
+		)
+		(instances
+			(project "12Board-PLC4UNI-G1W"
+				(path "/6879a69d-f695-48f8-b9bf-6eca45a0aeb9/dec84266-09cb-480d-928b-b373c3576401"
+					(page "32")
+				)
+			)

Commit message: actualizacion 76
Other:
- sheet output_4_20ma ports: added IN_mA, mA_out; removed Out_4-20mA
Changed lines of the file:
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@@
+	(wire
+		(pts
+			(xy 180.34 49.53) (xy 185.42 49.53)
+		)
+		(stroke
+			(width 0)
+			(type default)
+		)
+	)
 	(wire
 		(pts
@@
 	(wire
 		(pts
+			(xy 190.5 86.36) (xy 196.85 86.36)
+		)
+		(stroke
+			(width 0)
+			(type default)
+		)
+	)
+	(wire
+		(pts
 			(xy 48.26 133.35) (xy 57.15 133.35)
 		)
@@
 	(wire
 		(pts
+			(xy 151.13 49.53) (xy 154.94 49.53)
+		)
+		(stroke
+			(width 0)
+			(type default)
+		)
+	)
+	(wire
+		(pts
 			(xy 86.36 73.66) (xy 87.63 73.66)
 		)
@@
 	(wire
 		(pts
+			(xy 190.5 83.82) (xy 196.85 83.82)
+		)
+		(stroke
+			(width 0)
+			(type default)
+		)
+	)
+	(wire
+		(pts
 			(xy 151.13 139.7) (xy 154.94 139.7)
 		)
@@
 	(wire
 		(pts
+			(xy 191.77 72.39) (xy 198.12 72.39)
+		)
+		(stroke
+			(width 0)
+			(type default)
+		)
+	)
+	(wire
+		(pts
 			(xy 205.74 120.65) (xy 191.77 120.65)
 		)
@@
 	(wire
 		(pts
+			(xy 191.77 67.31) (xy 198.12 67.31)
+		)
+		(stroke
+			(width 0)
+			(type default)
+		)
+	)
+	(wire
+		(pts
 			(xy 53.34 142.24) (xy 58.42 142.24)
 		)
@@
 		(pts
 			(xy 78.74 168.91) (xy 87.63 168.91)
+		)
+		(stroke
+			(width 0)
+			(type default)
+		)
+	)
+	(wire
+		(pts
+			(xy 191.77 69.85) (xy 198.12 69.85)
 		)
 		(stroke
@@
 		)
 	)
+	(hierarchical_label "out-no-2"
+		(shape output)
+		(at 196.85 86.36 0)
+		(effects
+			(font
+				(size 1.27 1.27)
+			)
+			(justify left)
+		)
+	)
+	(hierarchical_label "mA_out1"
+		(shape output)
+		(at 185.42 49.53 0)
+		(effects
+			(font
+				(size 1.27 1.27)
+			)
+			(justify left)
+		)
+	)
 	(hierarchical_label "IN_0-10V"
 		(shape input)
@@
 		)
 	)
+	(hierarchical_label "out-common-2"
+		(shape output)
+		(at 196.85 83.82 0)
+		(effects
+			(font
+				(size 1.27 1.27)
+			)
+			(justify left)
+		)
+	)
+	(hierarchical_label "out-no-1"
+		(shape output)
+		(at 198.12 72.39 0)
+		(effects
+			(font
+				(size 1.27 1.27)
+			)
+			(justify left)
+		)
+	)
 	(hierarchical_label "NPN_OUT_Opto"
 		(shape output)
@@
 			)
 			(justify right)
+		)
+	)
+	(hierarchical_label "out-nc"
+		(shape output)
+		(at 198.12 69.85 0)
+		(effects
+			(font
+				(size 1.27 1.27)
+			)
+			(justify left)
+		)
+	)
+	(hierarchical_label "out-common-1"
+		(shape output)
+		(at 198.12 67.31 0)
+		(effects
+			(font
+				(size 1.27 1.27)
+			)
+			(justify left)
 		)
 	)
@@
 			)
 		)
-		(pin "Out_4-20mA" output
-			(at 180.34 50.8 0)
-			(effects
-				(font
+		(pin "IN_mA" input
+			(at 154.94 49.53 180)
+			(effects
+				(font
+					(size 1.27 1.27)
+				)
+				(justify left)
+			)
+		)
+		(pin "mA_out" output
+			(at 180.34 49.53 0)
+			(effects
+				(font
