File: diseños de kicad/12Board-PLC4UNI-G1W/entrada3.3v.kicad_sch (KiCad schematic)
At the start: 6 parts, among them U3 AP63203WU

Commit message: actualizacion 76
Parts:
- removed C4: 10uF, PCM_Capacitor_SMD_AKL:C_1206_3216Metric, symbol PCM_Capacitor_AKL:C_0603
- removed C5: 100nF, PCM_Capacitor_SMD_AKL:C_0805_2012Metric, symbol PCM_Capacitor_AKL:C_0603
- removed C6, C7: 22uF, PCM_Capacitor_SMD_AKL:C_1206_3216Metric, symbol PCM_Capacitor_AKL:C_0603
- removed L?: ANR4030T6R8M, Inductor_SMD:L_APV_ANR4030, symbol NR6028T4R7M:NR6028T4R7M
- removed U3: AP63203WU, Package_TO_SOT_SMD:TSOT-23-6, symbol Regulator_Switching:AP63203WU
- added C10: 100nF, PCM_Capacitor_SMD_AKL:C_0805_2012Metric, symbol PCM_Capacitor_AKL:C_0603
- added C11, C12: 22uF, PCM_Capacitor_SMD_AKL:C_1206_3216Metric, symbol PCM_Capacitor_AKL:C_0603
- added C9: 10uF, PCM_Capacitor_SMD_AKL:C_1206_3216Metric, symbol PCM_Capacitor_AKL:C_0603
- added F1: Fuse, Fuse:Fuse_1812_4532Metric, symbol Device:Fuse
- added L1: ANR4030T6R8M, Inductor_SMD:L_APV_ANR4030, symbol NR6028T4R7M:NR6028T4R7M
- added LED1: LED_0603_Red, PCM_LED_SMD_AKL:LED_0603_1608Metric, symbol PCM_LED_AKL:LED_0603_Red
- added R45: 1k, PCM_SparkFun-Resistor:R_0603_1608Metric, symbol PCM_SparkFun-Resistor:4.7k_0603
- added U4: AP63203WU, Package_TO_SOT_SMD:TSOT-23-6, symbol Regulator_Switching:AP63203WU
Connections:
- net GND: now also C11.2, C12.2, C9.2, LED1.1 (K), U4.4 (GND)
- new net: C10.1, U4.6 (BST)
- new net: C10.2, L1.1, U4.5 (SW)
- new net: LED1.2 (A), R45.1
- new net +24V: F1.1
- new net +3.3V: C11.1, C12.1, L1.2, U4.1 (FB)
- new net VCC: C9.1, F1.2, R45.2, U4.2 (EN), U4.3 (IN)
