File: diseños de kicad/12Board-PLC4UNI-G1W/out_put_relay1.kicad_sch (KiCad schematic)
At the start: 7 parts

Commit message: actualizacion 76
Parts:
- gave numbers to parts that had none: 3
Changed lines of the file:
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@@
 		(on_board yes)
 		(dnp no)
-		(property "Reference" "Q?"
+		(property "Reference" "Q11"
 			(at 157.48 99.0599 0)
 			(effects
@@
 			(project "12Board-PLC4UNI-G1W"
 				(path "/6879a69d-f695-48f8-b9bf-6eca45a0aeb9/dec84266-09cb-480d-928b-b373c3576401/85a80b9b-64d5-4833-b609-948fcc748275"
-					(reference "Q?")
+					(reference "Q11")
 					(unit 1)
 				)
@@
 		(on_board yes)
 		(dnp no)
-		(property "Reference" "OC?"
+		(property "Reference" "OC8"
 			(at 130.81 91.4399 0)
 			(effects
@@
 			(project "12Board-PLC4UNI-G1W"
 				(path "/6879a69d-f695-48f8-b9bf-6eca45a0aeb9/dec84266-09cb-480d-928b-b373c3576401/85a80b9b-64d5-4833-b609-948fcc748275"
-					(reference "OC?")
+					(reference "OC8")
 					(unit 1)
 				)
@@
 		(dnp no)
 		(fields_autoplaced yes)
-		(property "Reference" "K?"
+		(property "Reference" "K2"
 			(at 171.45 82.5499 0)
 			(effects
@@
 			(project "12Board-PLC4UNI-G1W"
 				(path "/6879a69d-f695-48f8-b9bf-6eca45a0aeb9/dec84266-09cb-480d-928b-b373c3576401/85a80b9b-64d5-4833-b609-948fcc748275"
-					(reference "K?")
-					(unit 1)
-				)
+					(reference "K2")
+					(unit 1)
+				)
