File: diseños de kicad/12Board-PLC4UNI-G1W/output_0_10v.kicad_sch (KiCad schematic)
At the start: 6 parts

Commit message: actualizacion 76
Parts:
- gave numbers to parts that had none: 5
Changed lines of the file:
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@@
 		(dnp no)
 		(fields_autoplaced yes)
-		(property "Reference" "C?"
+		(property "Reference" "C5"
 			(at 182.88 110.4899 0)
 			(effects
@@
 			(project "12Board-PLC4UNI-G1W"
 				(path "/6879a69d-f695-48f8-b9bf-6eca45a0aeb9/dec84266-09cb-480d-928b-b373c3576401/497cfd67-7ac2-4c40-abaf-60bdf8025b20"
-					(reference "C?")
+					(reference "C5")
 					(unit 1)
 				)
@@
 		(dnp no)
 		(fields_autoplaced yes)
-		(property "Reference" "R?"
+		(property "Reference" "R47"
 			(at 123.19 95.2499 90)
 			(effects
@@
 			(project "12Board-PLC4UNI-G1W"
 				(path "/6879a69d-f695-48f8-b9bf-6eca45a0aeb9/dec84266-09cb-480d-928b-b373c3576401/497cfd67-7ac2-4c40-abaf-60bdf8025b20"
-					(reference "R?")
+					(reference "R47")
 					(unit 1)
 				)
@@
 		(on_board yes)
 		(dnp no)
-		(property "Reference" "R?"
+		(property "Reference" "R46"
 			(at 110.49 95.25 90)
 			(effects
@@
 			(project "12Board-PLC4UNI-G1W"
 				(path "/6879a69d-f695-48f8-b9bf-6eca45a0aeb9/dec84266-09cb-480d-928b-b373c3576401/497cfd67-7ac2-4c40-abaf-60bdf8025b20"
-					(reference "R?")
+					(reference "R46")
 					(unit 1)
 				)
@@
 		(dnp no)
 		(fields_autoplaced yes)
-		(property "Reference" "U?"
+		(property "Reference" "U3"
 			(at 140.97 91.44 0)
 			(effects
@@
 			(project "12Board-PLC4UNI-G1W"
 				(path "/6879a69d-f695-48f8-b9bf-6eca45a0aeb9/dec84266-09cb-480d-928b-b373c3576401/497cfd67-7ac2-4c40-abaf-60bdf8025b20"
-					(reference "U?")
+					(reference "U3")
 					(unit 1)
 				)
@@
 		(dnp no)
 		(fields_autoplaced yes)
-		(property "Reference" "C?"
+		(property "Reference" "C4"
 			(at 162.56 93.98 90)
 			(effects
@@
 			(project "12Board-PLC4UNI-G1W"
 				(path "/6879a69d-f695-48f8-b9bf-6eca45a0aeb9/dec84266-09cb-480d-928b-b373c3576401/497cfd67-7ac2-4c40-abaf-60bdf8025b20"
-					(reference "C?")
-					(unit 1)
-				)
+					(reference "C4")
+					(unit 1)
+				)
