File: diseños de kicad/12Board-PLC4UNI-G1W/output_4_20ma.kicad_sch (KiCad schematic)
At the start: 0 parts

Commit message: actualizacion 3
Parts:
- added C8: 100nF, PCM_Capacitor_SMD_AKL:C_0603_1608Metric, symbol PCM_Capacitor_AKL:C_0603
- added R42: 120, PCM_Resistor_SMD_AKL:R_0603_1608Metric, symbol PCM_Resistor_AKL:R_0603
Connections:
- new net GND: C8.2, R42.2
- new net IN_mA: C8.1, R42.1

Commit message: actualizacion 76
Changed lines of the file:
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@@
-		)
-	)
-	(hierarchical_label "Out_4-20mA"
-		(shape output)
-		(at 127 97.79 0)
-		(effects
-			(font
-				(size 1.27 1.27)
-			)
-			(justify left)
 		)
 	)
