File: diseños de kicad/12Board-PLC4UNI-G1W/proteccion24.kicad_sch (KiCad schematic)
At the start: 6 parts

Commit message: actualizacion 76
Parts:
- gave numbers to parts that had none: 4
Changed lines of the file:
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@@
 		(on_board yes)
 		(dnp no)
-		(property "Reference" "F?"
+		(property "Reference" "F2"
 			(at 160.02 92.71 90)
 			(effects
@@
 			(project "12Board-PLC4UNI-G1W"
 				(path "/6879a69d-f695-48f8-b9bf-6eca45a0aeb9/dec84266-09cb-480d-928b-b373c3576401/dee64336-8ffb-410f-88f7-b3f5eafe9da9"
-					(reference "F?")
+					(reference "F2")
 					(unit 1)
 				)
@@
 		(on_board yes)
 		(dnp no)
-		(property "Reference" "LED?"
+		(property "Reference" "LED3"
 			(at 198.12 111.7599 90)
 			(effects
@@
 			(project "12Board-PLC4UNI-G1W"
 				(path "/6879a69d-f695-48f8-b9bf-6eca45a0aeb9/dec84266-09cb-480d-928b-b373c3576401/dee64336-8ffb-410f-88f7-b3f5eafe9da9"
-					(reference "LED?")
+					(reference "LED3")
 					(unit 1)
 				)
@@
 		(on_board yes)
 		(dnp no)
-		(property "Reference" "LED?"
+		(property "Reference" "LED2"
 			(at 147.32 111.7599 90)
 			(effects
@@
 			(project "12Board-PLC4UNI-G1W"
 				(path "/6879a69d-f695-48f8-b9bf-6eca45a0aeb9/dec84266-09cb-480d-928b-b373c3576401/dee64336-8ffb-410f-88f7-b3f5eafe9da9"
-					(reference "LED?")
+					(reference "LED2")
 					(unit 1)
 				)
@@
 		(on_board yes)
 		(dnp no)
-		(property "Reference" "RV?"
+		(property "Reference" "RV1"
 			(at 177.8 108.1432 0)
 			(effects
@@
 			(project "12Board-PLC4UNI-G1W"
 				(path "/6879a69d-f695-48f8-b9bf-6eca45a0aeb9/dec84266-09cb-480d-928b-b373c3576401/dee64336-8ffb-410f-88f7-b3f5eafe9da9"
-					(reference "RV?")
+					(reference "RV1")
 					(unit 1)
 				)
