File: diseños de kicad/12Board-PLC4UNI-G1W/rs485_protection.kicad_sch (KiCad schematic)
At the start: 1 part

Commit message: actualizacion 76
Parts:
- gave numbers to parts that had none: 1
Changed lines of the file:
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@@
 		(dnp no)
 		(fields_autoplaced yes)
-		(property "Reference" "#PWR?"
+		(property "Reference" "#PWR0101"
 			(at 149.86 113.03 0)
 			(effects
@@
 			(project "12Board-PLC4UNI-G1W"
 				(path "/6879a69d-f695-48f8-b9bf-6eca45a0aeb9/dec84266-09cb-480d-928b-b373c3576401/97147ee3-ae03-4b46-930a-a7427349894f/8cd41394-2f63-4fab-828d-268eea6a424c"
-					(reference "#PWR?")
+					(reference "#PWR0101")
 					(unit 1)
 				)
@@
 		(dnp no)
 		(fields_autoplaced yes)
-		(property "Reference" "D?"
+		(property "Reference" "D5"
 			(at 156.21 94.5514 90)
 			(effects
@@
 			(project "12Board-PLC4UNI-G1W"
 				(path "/6879a69d-f695-48f8-b9bf-6eca45a0aeb9/dec84266-09cb-480d-928b-b373c3576401/97147ee3-ae03-4b46-930a-a7427349894f/8cd41394-2f63-4fab-828d-268eea6a424c"
-					(reference "D?")
+					(reference "D5")
 					(unit 1)
 				)
