File: diseños de kicad/12Board-PLC4UNI-G1W/12Board-PLC4UNI-G1W.kicad_pcb (KiCad board)
At the start: 2 copper layers, 0 parts

Commit message: actualizacion 76
Parts:
- added D2: 1N4148WT, Diode_SMD:D_SOD-523, F.Cu at (125.1, 112.2)
- added D3: 1N4148WT, Diode_SMD:D_SOD-523, F.Cu at (129.4, 121.5)
- added D4: SMF24A, Diode_SMD:D_SMF, F.Cu at (134.9, 94.0)
- added F1: Fuse, Fuse:Fuse_1812_4532Metric, F.Cu at (125.9, 106.3)
- added F2: Fuse, Fuse:Fuse_0603_1608Metric, F.Cu at (157.1, 67.6)
- added K1: Fujitsu_FTR-LYAA005x, Relay_THT:Relay_SPST-NO_Fujitsu_FTR-LYAA005x_FormA_Vertical, F.Cu at (127.0, 125.2)
- added K2: Fujitsu_FTR-LYCA005x, Relay_THT:Relay_SPDT_Fujitsu_FTR-LYCA005x_FormC_Vertical, F.Cu at (126.9, 118.3)
- added L1: ANR4030T6R8M, Inductor_SMD:L_APV_ANR4030, F.Cu at (129.4, 98.7)
- added R1: R_US, Resistor_SMD:R_0201_0603Metric, F.Cu at (137.3, 109.0)
- added R2: R_US, Resistor_SMD:R_0201_0603Metric, F.Cu at (136.9, 110.5)
- added RV1: Varistor, Varistor:RV_Disc_D7mm_W3.4mm_P5mm, F.Cu at (153.3, 68.2)
- added U1: ESP32-S3-WROOM-1, RF_Module:ESP32-S3-WROOM-1, F.Cu at (147.9, 99.0)
- added U4: AP63203WU, Package_TO_SOT_SMD:TSOT-23-6, F.Cu at (134.8, 97.7)
- added connector-up1: Screw_Terminal_9_P5.00mm, TerminalBlock_Phoenix:TerminalBlock_Phoenix_PT-1,5-9-5.0-H_1x09_P5.00mm_Horizontal, F.Cu at (102.8, 59.6)
- added connector-up2: Screw_Terminal_9_P5.00mm, TerminalBlock_Phoenix:TerminalBlock_Phoenix_PT-1,5-9-5.0-H_1x09_P5.00mm_Horizontal, F.Cu at (149.8, 59.2)
- added connector-up3: Screw_Terminal_9_P5.00mm, TerminalBlock_Phoenix:TerminalBlock_Phoenix_PT-1,5-9-5.0-H_1x09_P5.00mm_Horizontal, F.Cu at (189.1, 133.8)
- added connector-up4: Screw_Terminal_9_P5.00mm, TerminalBlock_Phoenix:TerminalBlock_Phoenix_PT-1,5-9-5.0-H_1x09_P5.00mm_Horizontal, F.Cu at (103.0, 132.9)
Routing:
- net GND: track 0.00 -> 86.9 mm
- net /board-plc4uni-G1w/out-no-1: track 0.00 -> 59.8 mm
- net VCC: track 0.00 -> 39.6 mm
- net /board-plc4uni-G1w/out-nc: track 0.00 -> 17.2 mm
- net /board-plc4uni-G1w/out-common-1: track 0.00 -> 16.7 mm
- net +3.3V: track 0.00 -> 12.3 mm
- net /board-plc4uni-G1w/out-common-2: track 0.00 -> 11.5 mm
- net /board-plc4uni-G1w/24V-SOURCE: track 0.00 -> 9.61 mm
- net /board-plc4uni-G1w/out-no-2: track 0.00 -> 9.01 mm
- net /board-plc4uni-G1w/0V-SOURCE: track 0.00 -> 8.24 mm
- net Net-(D2-A): track 0.00 -> 7.65 mm
- net Net-(U4-SW): track 0.00 -> 7.55 mm
- net Net-(D3-A): track 0.00 -> 7.02 mm
- net Net-(F2-Pad1): track 0.00 -> 3.24 mm
- net /board-plc4uni-G1w/plc4uni_cpu/USB+: track 0.00 -> 1.97 mm
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
Commit message: actualizacion 45
Parts:
- added C1: 100nF, Capacitor_SMD:C_0201_0603Metric, F.Cu at (215.3, 93.2)
- added C10: 1uF, Capacitor_SMD:C_0805_2012Metric, F.Cu at (204.6, 71.3)
- added C11: 10uF, PCM_Capacitor_SMD_AKL:C_1206_3216Metric, F.Cu at (302.2, 58.5)
- added C12: 100nF, PCM_Capacitor_SMD_AKL:C_0805_2012Metric, F.Cu at (310.4, 53.8)
- added C13: 22uF, PCM_Capacitor_SMD_AKL:C_1206_3216Metric, F.Cu at (306.2, 62.8)
- added C14: 22uF, PCM_Capacitor_SMD_AKL:C_1206_3216Metric, F.Cu at (306.2, 60.0)
- added C2: 0.1uF, PCM_Capacitor_SMD_AKL:C_0603_1608Metric, F.Cu at (346.9, 55.8)
- added C3: 1uF, PCM_Capacitor_SMD_AKL:C_0603_1608Metric, F.Cu at (374.9, 106.9)
- added C4: 0.1uF, PCM_Capacitor_SMD_AKL:C_0603_1608Metric, F.Cu at (371.6, 107.6)
- added C5: 220pF, Capacitor_SMD:C_0805_2012Metric, F.Cu at (204.6, 81.3)
- added C6: 1uF, Capacitor_SMD:C_0805_2012Metric, F.Cu at (204.6, 84.3)
- added C7: 1uF, Capacitor_SMD:C_0805_2012Metric, F.Cu at (204.6, 87.3)
- added C8: 220pF, Capacitor_SMD:C_0805_2012Metric, F.Cu at (204.6, 65.3)
- added C9: 1uF, Capacitor_SMD:C_0805_2012Metric, F.Cu at (204.6, 68.3)
- added D1: TVA, PCM_Diode_SMD_AKL:D_SOD-123F, F.Cu at (372.4, 110.0)
- added D10: D_Zener, Diode_SMD:D_0603_1608Metric, F.Cu at (212.9, 74.9)
- added D11: SMF24A, Diode_SMD:D_SMF, F.Cu at (213.7, 71.9)
- added D2: D_Zener, Diode_SMD:D_0603_1608Metric, F.Cu at (212.9, 90.9)
- added D3: SMF24A, Diode_SMD:D_SMF, F.Cu at (213.7, 87.9)
- added D5: 1N4148WT, Diode_SMD:D_SOD-523, F.Cu at (340.0, 105.0)
- added D6: 1N4148WT, Diode_SMD:D_SOD-523, F.Cu at (350.1, 104.6)
- added D7: M7, PCM_Diode_SMD_AKL:D_SMA, F.Cu at (326.8, 107.4)
- added D8: M7, PCM_Diode_SMD_AKL:D_SMA, F.Cu at (318.6, 107.8)
- added D9: M7, PCM_Diode_SMD_AKL:D_SMA, F.Cu at (335.7, 107.6)
- added F1: Fuse, Fuse:Fuse_1812_4532Metric, F.Cu at (301.9, 52.0)
- added K1: G5V-1, Relay_THT:Relay_SPDT_Omron_G5V-1, F.Cu at (342.5, 99.9)
- added K2: G5V-1, Relay_THT:Relay_SPDT_Omron_G5V-1, F.Cu at (352.6, 99.9)
- added L1: ANR4030T6R8M, Inductor_SMD:L_APV_ANR4030, F.Cu at (311.2, 57.5)
- added LED1: LED_0603_Red, PCM_LED_SMD_AKL:LED_0603_1608Metric, F.Cu at (299.4, 43.8)
- added OC1: TLP293, PCM_Package_SO_AKL:SOP-4_4.4x2.6mm_P1.27mm, F.Cu at (340.5, 55.4)
- added OC2: TLP293, PCM_Package_SO_AKL:SOP-4_4.4x2.6mm_P1.27mm, F.Cu at (372.8, 55.5)
- added OC3: TLP293, PCM_Package_SO_AKL:SOP-4_4.4x2.6mm_P1.27mm, F.Cu at (335.8, 55.5)
- added OC4: TLP293, PCM_Package_SO_AKL:SOP-4_4.4x2.6mm_P1.27mm, F.Cu at (367.6, 55.5)
- added Q10: BC817, PCM_Package_TO_SOT_SMD_AKL:SOT-23, F.Cu at (326.8, 99.7)
- added Q11: MMBT4403, PCM_Package_TO_SOT_SMD_AKL:SOT-23, F.Cu at (322.8, 106.8)
- added Q12: BC817, PCM_Package_TO_SOT_SMD_AKL:SOT-23, F.Cu at (318.5, 100.1)
- added Q13: MMBT4403, PCM_Package_TO_SOT_SMD_AKL:SOT-23, F.Cu at (313.6, 106.5)
- added Q14: BC817, PCM_Package_TO_SOT_SMD_AKL:SOT-23, F.Cu at (335.6, 100.1)
- added Q15: MMBT4403, PCM_Package_TO_SOT_SMD_AKL:SOT-23, F.Cu at (331.5, 108.5)
- added Q2: BC817, PCM_Package_TO_SOT_SMD_AKL:SOT-23, F.Cu at (330.7, 51.3)
- added Q3: BC817, PCM_Package_TO_SOT_SMD_AKL:SOT-23, F.Cu at (362.5, 51.0)
- added Q4: BC817, PCM_Package_TO_SOT_SMD_AKL:SOT-23, F.Cu at (323.7, 51.3)
- added Q5: BC817, PCM_Package_TO_SOT_SMD_AKL:SOT-23, F.Cu at (385.2, 109.6)
- added Q6: BC817, PCM_Package_TO_SOT_SMD_AKL:SOT-23, F.Cu at (352.4, 50.8)
- added Q7: BC817, PCM_Package_TO_SOT_SMD_AKL:SOT-23, F.Cu at (347.0, 96.5)
- added Q8: BC817, PCM_Package_TO_SOT_SMD_AKL:SOT-23, F.Cu at (357.2, 96.5)
- added Q9: BC817, PCM_Package_TO_SOT_SMD_AKL:SOT-23, F.Cu at (381.4, 109.6)
- added R1: 10k, PCM_Resistor_SMD_AKL:R_0603_1608Metric, F.Cu at (316.0, 81.8)
- added R10: 470, PCM_SparkFun-Resistor:R_0603_1608Metric, F.Cu at (268.1, 30.2)
- added R11: 470, PCM_SparkFun-Resistor:R_0603_1608Metric, F.Cu at (264.3, 54.1)
- added R12: 20K, PCM_Resistor_SMD_AKL:R_0603_1608Metric, F.Cu at (344.9, 52.5)
- added R13: 10K, PCM_Resistor_SMD_AKL:R_0603_1608Metric, F.Cu at (344.9, 55.7)
- added R14: 4.7k, PCM_Resistor_SMD_AKL:R_0603_1608Metric, F.Cu at (373.8, 97.5)
- added R15: 4.7k, PCM_Resistor_SMD_AKL:R_0603_1608Metric, F.Cu at (371.9, 97.5)
- added R16: 2.5k, PCM_Resistor_SMD_AKL:R_0603_1608Metric, F.Cu at (263.9, 79.5)
- added R17: 470k, PCM_Resistor_SMD_AKL:R_0603_1608Metric, F.Cu at (263.9, 82.2)
- added R18: 15, PCM_Resistor_SMD_AKL:R_0603_1608Metric, F.Cu at (263.9, 84.9)
- added R19: 10K, PCM_Resistor_SMD_AKL:R_0603_1608Metric, F.Cu at (335.8, 50.0)
- added R2: 10k, PCM_Resistor_SMD_AKL:R_0603_1608Metric, F.Cu at (316.0, 84.5)
- added R20: 10K, PCM_Resistor_SMD_AKL:R_0603_1608Metric, F.Cu at (335.8, 60.8)
- added R21: 10K, PCM_Resistor_SMD_AKL:R_0603_1608Metric, F.Cu at (327.2, 50.3)
- added R22: 2.4K, PCM_Resistor_SMD_AKL:R_0603_1608Metric, F.Cu at (331.0, 54.0)
- added R23: 4.7K, PCM_Resistor_SMD_AKL:R_0603_1608Metric, F.Cu at (367.6, 50.0)
- added R24: 2.4K, PCM_Resistor_SMD_AKL:R_0603_1608Metric, F.Cu at (367.8, 60.9)
- added R25: 10K, PCM_Resistor_SMD_AKL:R_0603_1608Metric, F.Cu at (358.8, 50.0)
- added R26: 47K, PCM_Resistor_SMD_AKL:R_0603_1608Metric, F.Cu at (358.7, 52.0)
- added R27: 2.4K, PCM_Resistor_SMD_AKL:R_0603_1608Metric, F.Cu at (362.7, 54.0)
- added R28: 10K, PCM_Resistor_SMD_AKL:R_0603_1608Metric, F.Cu at (320.2, 50.3)
- added R29: 2.4K, PCM_Resistor_SMD_AKL:R_0603_1608Metric, F.Cu at (323.9, 54.0)
- added R3: 10k, PCM_Resistor_SMD_AKL:R_0603_1608Metric, F.Cu at (316.0, 87.2)
- added R30: 2.4k, PCM_Resistor_SMD_AKL:R_0603_1608Metric, F.Cu at (388.0, 107.5)
- added R31: 10k, PCM_Resistor_SMD_AKL:R_0603_1608Metric, F.Cu at (385.5, 106.6)
- added R32: 10K, PCM_Resistor_SMD_AKL:R_0603_1608Metric, F.Cu at (348.8, 49.8)
- added R33: 47K, PCM_Resistor_SMD_AKL:R_0603_1608Metric, F.Cu at (348.8, 51.5)
- added R34: 2.4K, PCM_Resistor_SMD_AKL:R_0603_1608Metric, F.Cu at (352.6, 53.5)
- added R35: 2.4k, PCM_Resistor_SMD_AKL:R_0603_1608Metric, F.Cu at (347.2, 93.5)
- added R36: 2.4k, PCM_Resistor_SMD_AKL:R_0603_1608Metric, F.Cu at (357.5, 93.6)
- added R37: 2.4k, PCM_Resistor_SMD_AKL:R_0603_1608Metric, F.Cu at (379.1, 106.7)
- added R38: 10k, PCM_Resistor_SMD_AKL:R_0603_1608Metric, F.Cu at (378.4, 109.2)
- added R39: 2.4k, PCM_Resistor_SMD_AKL:R_0603_1608Metric, F.Cu at (328.8, 96.8)
- added R4: 10k, PCM_Resistor_SMD_AKL:R_0603_1608Metric, F.Cu at (257.8, 89.6)
- added R40: 10k, PCM_Resistor_SMD_AKL:R_0603_1608Metric, F.Cu at (329.7, 99.6)
- added R41: 4.7k, PCM_Resistor_SMD_AKL:R_0603_1608Metric, F.Cu at (326.9, 102.6)
- added R42: 10k, PCM_Resistor_SMD_AKL:R_0603_1608Metric, F.Cu at (323.4, 102.7)
- added R43: 10k, PCM_Resistor_SMD_AKL:R_0603_1608Metric, F.Cu at (322.8, 109.7)
- added R44: 2.4k, PCM_Resistor_SMD_AKL:R_0603_1608Metric, F.Cu at (318.8, 97.3)
- added R45: 10k, PCM_Resistor_SMD_AKL:R_0603_1608Metric, F.Cu at (315.4, 99.8)
- added R46: 4.7k, PCM_Resistor_SMD_AKL:R_0603_1608Metric, F.Cu at (311.2, 109.4)
- added R47: 10k, PCM_Resistor_SMD_AKL:R_0603_1608Metric, F.Cu at (318.4, 103.1)
- added R48: 10k, PCM_Resistor_SMD_AKL:R_0603_1608Metric, F.Cu at (314.5, 109.3)
- added R49: 2.4k, PCM_Resistor_SMD_AKL:R_0603_1608Metric, F.Cu at (337.7, 97.2)
- added R5: 10k, PCM_Resistor_SMD_AKL:R_0603_1608Metric, F.Cu at (257.8, 92.3)
- added R50: 10k, PCM_Resistor_SMD_AKL:R_0603_1608Metric, F.Cu at (338.4, 99.7)
- added R51: 4.7k, PCM_Resistor_SMD_AKL:R_0603_1608Metric, F.Cu at (335.7, 102.9)
- added R52: 10k, PCM_Resistor_SMD_AKL:R_0603_1608Metric, F.Cu at (331.9, 104.4)
- added R53: 10k, PCM_Resistor_SMD_AKL:R_0603_1608Metric, F.Cu at (338.8, 109.7)
- added R54: 2.5k, PCM_Resistor_SMD_AKL:R_0603_1608Metric, F.Cu at (257.8, 79.5)
- added R55: 470k, PCM_Resistor_SMD_AKL:R_0603_1608Metric, F.Cu at (257.8, 82.2)
- added R56: 15, PCM_Resistor_SMD_AKL:R_0603_1608Metric, F.Cu at (257.8, 84.9)
- added R57: 1k, PCM_SparkFun-Resistor:R_0603_1608Metric, F.Cu at (300.1, 46.5)
- added R6: 10K, PCM_Resistor_SMD_AKL:R_0603_1608Metric, F.Cu at (340.5, 50.1)
- added R7: 10K, PCM_Resistor_SMD_AKL:R_0603_1608Metric, F.Cu at (340.6, 60.7)
- added R8: 4.7K, PCM_Resistor_SMD_AKL:R_0603_1608Metric, F.Cu at (372.8, 50.0)
- added R9: 2.4K, PCM_Resistor_SMD_AKL:R_0603_1608Metric, F.Cu at (372.8, 60.8)
- added U1: SP3485EN, Package_SO:SOIC-8_3.9x4.9mm_P1.27mm, F.Cu at (322.2, 84.3)
- added U4: ~, Lib_GP8211S-TC50-EW:ESOP-8_L4.9-W3.9-P1.27-LS6.0-BL-EP, F.Cu at (371.6, 102.9)
- added U5: ~, Package_SO:SSOP-10-1EP_3.9x4.9mm_P1mm_EP2.1x3.3mm, F.Cu at (211.4, 83.0)
- added U6: ~, Package_SO:SSOP-10-1EP_3.9x4.9mm_P1mm_EP2.1x3.3mm, F.Cu at (211.4, 67.0)
- added U7: AP63203WU, Package_TO_SOT_SMD:TSOT-23-6, F.Cu at (306.3, 56.1)
- added U8: ESP32-S3-MINI-1U, RF_Module:ESP32-S2-MINI-1U, F.Cu at (383.9, 79.3)
- moved RV1 63.0 mm to (94.3, 46.0)
- moved D2 63.0 mm to (66.1, 90.0)
- moved F1 63.0 mm to (66.9, 84.1)
- moved F2 63.0 mm to (98.1, 45.4)
- moved K1 63.0 mm to (68.0, 103.0)
- moved K2 63.0 mm to (67.9, 96.1)
- moved L1 63.0 mm to (70.4, 76.5)
- moved R1 63.0 mm to (78.3, 86.8)
- moved U1 63.0 mm to (88.9, 76.8)
- moved U4 63.0 mm to (75.8, 75.5)
- moved connector-up1 63.0 mm to (43.8, 37.5)
- moved connector-up2 63.0 mm to (90.8, 37.1)
- moved connector-up3 63.0 mm to (130.1, 111.7)
- moved connector-up4 63.0 mm to (44.0, 110.7)
- moved D3 63.0 mm to (70.5, 99.4)
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Routing:
- net GND: track 86.9 -> 250.4 mm, vias 0 -> 16
- net +3.3V: track 12.3 -> 126.7 mm
- net VCC: track 39.6 -> 87.2 mm
- net /Board-PLC4UNI-G1W/out-no-2: track 0.00 -> 21.7 mm
- net Net-(D6-A): track 0.00 -> 17.4 mm
- net Net-(D5-A): track 0.00 -> 17.2 mm
- net Net-(Q12-C): track 0.00 -> 16.1 mm
- net /Board-PLC4UNI-G1W/PNP_OUT3: track 0.00 -> 16.1 mm
- net /Board-PLC4UNI-G1W/out-common-1: track 0.00 -> 15.1 mm
- net /Board-PLC4UNI-G1W/PNP_OUT2: track 0.00 -> 13.9 mm
- net /Board-PLC4UNI-G1W/PNP_OUT1: track 0.00 -> 13.7 mm
- net /Board-PLC4UNI-G1W/out-common-2: track 0.00 -> 12.0 mm
- net Net-(Q12-B): track 0.00 -> 11.3 mm
- net /Board-PLC4UNI-G1W/Out_0-10V: track 0.00 -> 10.8 mm
- net /Board-PLC4UNI-G1W/NPN_OUT1: track 0.00 -> 9.91 mm
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- added copper zone on F.Cu, net +3.3V
- added copper zone on F.Cu, net GND
- added copper zone on F.Cu, net Net-(U7-SW)
Other:
- board outline added: 100 x 80.2 mm

Commit message: actualizacion 234
Parts:
- removed the D2 at (66.1, 90.0)
- removed the D3 at (70.5, 99.4)
- removed D4: SMF24A, Diode_SMD:D_SMF
- removed the F1 at (66.9, 84.1)
- removed F2: Fuse, Fuse:Fuse_0603_1608Metric
- removed the K1 at (68.0, 103.0)
- removed the K2 at (67.9, 96.1)
- removed the L1 at (70.4, 76.5)
- removed the R1 at (78.3, 86.8)
- removed the R2 at (78.0, 88.3)
- removed RV1: Varistor, Varistor:RV_Disc_D7mm_W3.4mm_P5mm
- removed the U1 at (88.9, 76.8)
- removed the U4 at (75.8, 75.5)
- moved C1 146.4 mm to (69.2, 103.6)
- moved C13 146.4 mm to (160.1, 73.2)
- moved C2 146.4 mm to (200.8, 66.2)
- moved C3 146.4 mm to (228.8, 117.3)
- moved C4 146.4 mm to (225.6, 118.0)
- moved D5 146.4 mm to (193.9, 115.4)
- moved D8 146.4 mm to (172.6, 118.2)
- moved D9 146.4 mm to (189.6, 118.0)
- moved K1 146.4 mm to (196.4, 110.3)
- moved OC3 146.4 mm to (189.8, 65.8)
- moved OC4 146.4 mm to (221.6, 65.9)
- moved Q10 146.4 mm to (180.8, 110.0)
- moved Q11 146.4 mm to (176.8, 117.2)
- moved Q13 146.4 mm to (167.6, 117.0)
- moved Q15 146.4 mm to (185.4, 119.0)
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Routing:
- net GND: track 250.4 -> 163.6 mm
- net /board-plc4uni-G1w/out-no-1: track 59.8 -> 0.00 mm
- net VCC: track 87.2 -> 47.7 mm
- net /board-plc4uni-G1w/out-nc: track 17.2 -> 0.00 mm
- net /board-plc4uni-G1w/out-common-1: track 16.7 -> 0.00 mm
- net +3.3V: track 126.7 -> 114.5 mm
- net /board-plc4uni-G1w/out-common-2: track 11.5 -> 0.00 mm
- net /board-plc4uni-G1w/24V-SOURCE: track 9.61 -> 0.00 mm
- net /board-plc4uni-G1w/out-no-2: track 9.01 -> 0.00 mm
- net /board-plc4uni-G1w/0V-SOURCE: track 8.24 -> 0.00 mm
- net Net-(D2-A): track 7.65 -> 0.00 mm
- net Net-(U4-SW): track 7.55 -> 0.00 mm
- net Net-(D3-A): track 7.02 -> 0.00 mm
- net Net-(F2-Pad1): track 3.24 -> 0.00 mm
- net /board-plc4uni-G1w/plc4uni_cpu/USB+: track 1.97 -> 0.00 mm
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
Commit message: actualizacion 234
Parts:
- removed R10, R11: 470, PCM_SparkFun-Resistor:R_0603_1608Metric
- removed R4, R5: 10k, PCM_Resistor_SMD_AKL:R_0603_1608Metric
- added J6: PINHD_2x5_Male, Connector_PinHeader_2.54mm:PinHeader_2x05_P2.54mm_Horizontal, F.Cu at (109.5, 97.0)
- moved C6 137.0 mm to (194.4, 112.2), turned to 180 degrees
- moved C5 134.5 mm to (190.9, 115.4), turned to 180 degrees
- moved C7 132.0 mm to (190.5, 101.9)
- moved U5 128.5 mm to (193.2, 107.2), turned to -90 degrees
- moved D3 124.6 mm to (190.3, 120.3), turned to 90 degrees
- moved D2 122.7 mm to (189.4, 105.1), turned to -90 degrees
- moved C10 111.8 mm to (169.3, 96.5), turned to 180 degrees
- moved C9 110.9 mm to (166.3, 104.8), turned to 90 degrees
- moved U6 109.4 mm to (171.6, 103.5), turned to 180 degrees
- moved C8 107.8 mm to (163.3, 101.0), turned to 90 degrees
- moved D10 107.5 mm to (173.3, 99.8), turned to 180 degrees
- moved D11 97.7 mm to (162.6, 105.3), turned to -90 degrees
- moved R17 79.9 mm to (193.1, 119.4)
- moved R18 79.6 mm to (193.1, 121.4), turned to 180 degrees
- moved R16 76.5 mm to (191.0, 112.2), turned to 180 degrees
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Connections:
- U8 pad 12: unconnected-(U8-IO8-Pad12) -> /Board-PLC4UNI-G1W/Output_0-10V/SDA
- U8 pad 13: unconnected-(U8-IO9-Pad13) -> /Board-PLC4UNI-G1W/Output_0-10V/SCL
- U8 pad 23: unconnected-(U8-USB_D--Pad23) -> /Board-PLC4UNI-G1W/PLC4UNI/USB-
- U8 pad 24: unconnected-(U8-USB_D+-Pad24) -> /Board-PLC4UNI-G1W/PLC4UNI/USB+
- U8 pad 25: unconnected-(U8-IO21-Pad25) -> /Board-PLC4UNI-G1W/Input_NPN1/OUT
- U8 pad 26: unconnected-(U8-IO26-Pad26) -> /Board-PLC4UNI-G1W/Input_NPN/OUT
- U8 pad 27: unconnected-(U8-IO47-Pad27) -> /Board-PLC4UNI-G1W/Output_NPN_Opto1/IN
- U8 pad 28: unconnected-(U8-IO33-Pad28) -> /Board-PLC4UNI-G1W/Input_PNP1_Opto/OUT
- U8 pad 29: unconnected-(U8-IO34-Pad29) -> /Board-PLC4UNI-G1W/Input_PNP2_Opto/OUT
- U8 pad 30: unconnected-(U8-IO48-Pad30) -> /Board-PLC4UNI-G1W/OutputRelay1/IN
- U8 pad 31: unconnected-(U8-IO35-Pad31) -> /Board-PLC4UNI-G1W/Input_NPN1_Opto/OUT
- U8 pad 32: unconnected-(U8-IO36-Pad32) -> /Board-PLC4UNI-G1W/Input_NPN1_Opto1/OUT
- U8 pad 33: unconnected-(U8-IO37-Pad33) -> /Board-PLC4UNI-G1W/Input_PNP/OUT
- U8 pad 34: unconnected-(U8-IO38-Pad34) -> /Board-PLC4UNI-G1W/Input_PNP2/OUT
- U8 pad 35: unconnected-(U8-IO39-Pad35) -> /Board-PLC4UNI-G1W/PLC4UNI/Out_4-20mA
- U8 pad 36: unconnected-(U8-IO40-Pad36) -> /Board-PLC4UNI-G1W/PLC4UNI/Out_4-20mA_2
- U8 pad 37: unconnected-(U8-IO41-Pad37) -> /Board-PLC4UNI-G1W/Output_PNP/IN
- U8 pad 38: unconnected-(U8-IO42-Pad38) -> /Board-PLC4UNI-G1W/Output_PNP1/IN
- U8 pad 4: unconnected-(U8-IO0-Pad4) -> /Board-PLC4UNI-G1W/Output_NPN1/IN
- U8 pad 41: unconnected-(U8-IO45-Pad41) -> /Board-PLC4UNI-G1W/Output_PNP2/IN
- U8 pad 44: unconnected-(U8-IO46-Pad44) -> /Board-PLC4UNI-G1W/Output_NPN_Opto/IN
- U8 pad 5: unconnected-(U8-IO1-Pad5) -> /Board-PLC4UNI-G1W/Output_NPN/IN
- U8 pad 6: unconnected-(U8-IO2-Pad6) -> /Board-PLC4UNI-G1W/OutRelay2/IN
- U8 pad 7: unconnected-(U8-IO3-Pad7) -> /Board-PLC4UNI-G1W/PLC4UNI/IN_4-20mA
- U8 pad 8: unconnected-(U8-IO4-Pad8) -> /Board-PLC4UNI-G1W/PLC4UNI/IN_4-20mA_2
- U8 pad 9: unconnected-(U8-IO5-Pad9) -> /Board-PLC4UNI-G1W/PLC4UNI/micro1_rs485_control
Routing:
- net VCC: track 47.7 -> 217.0 mm, vias 0 -> 14
- net GND: track 163.6 -> 279.6 mm, vias 16 -> 28
- net /Board-PLC4UNI-G1W/PLC4UNI/micro_rs485_tx: track 0.00 -> 84.4 mm
- net /Board-PLC4UNI-G1W/PLC4UNI/micro_rs485_rx: track 0.00 -> 83.5 mm, vias 0 -> 2
- net /Board-PLC4UNI-G1W/Output_0-10V/SDA: track 1.76 -> 51.2 mm, vias 0 -> 2
- net /Board-PLC4UNI-G1W/con_RS485_B: track 0.00 -> 44.4 mm
- net /Board-PLC4UNI-G1W/Output_0-10V/SCL: track 1.74 -> 35.9 mm
- net +3.3V: track 114.5 -> 146.0 mm, vias 0 -> 6
- net /Board-PLC4UNI-G1W/con_RS485_A: track 0.00 -> 29.0 mm
- net Net-(D2-A): track 0.00 -> 24.6 mm
- net Net-(U6-SET): track 0.00 -> 5.84 mm
- net Net-(U5-SET): track 0.00 -> 5.76 mm
- net Net-(D10-A): track 0.00 -> 5.67 mm
- net Net-(D11-A1): track 0.00 -> 3.52 mm
- net Net-(U6-V5V): track 0.00 -> 2.67 mm
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Other:
- outline, holes or cut-outs redrawn

Commit message: actualizacion23
Routing:
- net +3.3V: track 146.0 -> 157.4 mm
Changed lines of the file:
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@@
+	)
+	(segment
+		(start 121.775 66.225)
+		(end 120.22 67.78)
+		(width 0.6)
+		(layer "F.Cu")
+		(net 39)
 	)
 	(segment
@@
 		(start 134.05 73.55)
 		(end 137.05 73.55)
-		(width 0.6)
-		(layer "F.Cu")
-		(net 39)
-	)
-	(segment
-		(start 116.795 67.78)
-		(end 114.495 67.78)
 		(width 0.6)
 		(layer "F.Cu")
@@
 	)
 	(segment
+		(start 120.22 67.78)
+		(end 114.495 67.78)
+		(width 0.6)
+		(layer "F.Cu")
+		(net 39)
+	)
+	(segment
 		(start 172.45 108.175)
 		(end 173.225 108.175)
@@
 	)
 	(segment
+		(start 112.495 74.03)
+		(end 108.725 77.8)
+		(width 0.6)
+		(layer "B.Cu")
+		(net 39)
+	)
+	(segment
 		(start 112.495 72.53)
 		(end 112.495 74.03)
@@
 	)
 	(segment
-		(start 112.495 74.03)
-		(end 111.495 75.03)
-		(width 0.6)
-		(layer "B.Cu")
-		(net 39)
-	)
-	(segment
 		(start 100.35 84.3)
 		(end 100.35 88.05)
@@
 		(width 0.6)
 		(layer "B.Cu")
+		(net 39)
+	)
+	(segment
+		(start 108.725 77.8)
+		(end 106.85 77.8)
+		(width 0.6)
+		(layer "B.Cu")
